File: pe/kicad-template/template.kicad_sch (KiCad schematic)
At the start: 0 parts

Commit message: push1
Parts:
- added C1: C, Package_SO:SOIC-8_3.9x4.9mm_P1.27mm, symbol Device:C
- added C2, C3, C4: C, symbol Device:C
- added L1: L, symbol Device:L
- added R1, R2: R, symbol Device:R
- added U1: TPS54302, Package_TO_SOT_SMD:SOT-23-6, symbol Regulator_Switching:TPS54302
Connections:
- new net: C1.2, U1.2 (SW)
- new net GND: U1.6 (BOOT)

Commit message: Move power electronics onboarding PDF to pe folder
Connections:
- net GND: now also R1.2
- net VCC: now also C3.2, R2.1, U1.3 (VIN), U1.5 (EN)
- net at C1.1: now also C3.1, L1.2
- net at L1.1: no longer names the net of L1.1
- net at L1.1: now also U1.4 (FB)
- net at R1.1: now also R2.2
Other:
- moved on the sheet: C3, R1, R2
